File: SmallKat Pressure Sensors.sch (KiCad schematic (older format))
At the start: 7 parts, among them J1 Conn_01x04_Male, U1 LPS25HB

Commit message: updated to single sided assembly
Parts:
- C1: value C -> 0.1uF
Connections:
- no-connect marks 0 -> 2
Changed lines of the file:
@@
 P 3400 1500
 F 0 "C1" H 3515 1546 50  0000 L CNN
-F 1 "C" H 3515 1455 50  0000 L CNN
+F 1 "0.1uF" H 3515 1455 50  0000 L CNN
 F 2 "Capacitor_SMD:C_0402_1005Metric" H 3438 1350 50  0001 C CNN
 F 3 "~" H 3400 1500 50  0001 C CNN
@@
 	1    0    0    -1
 $EndComp
+NoConn ~ 3850 2250
+NoConn ~ 3850 2450
 $EndSCHEMATC
